File: board/turret.kicad_sch (KiCad schematic)
At the start: 54 parts, among them M1 SRV_LAS, M2 SRV_SEN, Q1 BC848, SW1 SW_Push, U1 STM32F103CBTx, U2 W25Q16JLSSIG, U3 TPA2005D1DGN, U4 TPS61322xADBV, U5 TLV70028_SOT23-5

Commit message: Board layout complete
Parts:
- removed H5, H6, H7: MountingHole_Pad, MountingHole:MountingHole_2.2mm_M2_DIN965_Pad, symbol Mechanical:MountingHole_Pad
Connections:
- net GND is gone; now on net GNDA: H4.1
- net VDD: now also C5.1
Other:
- moved on the sheet: C5
